File: Audio&PowerDaughterboard/Audio&Power DB.kicad_pcb (KiCad board)
At the start: 2 copper layers, 30 x 108 mm, 20 parts, among them J1 AudioJack3, J2 AudioJack3, J3 AudioJack3, J4 USB_C_Receptacle_USB2.0, J5 Conn_01x09, U1 SGTL5000XNLA3, U2 NCP1117-3.3_SOT223, U3 AP2127N-1.2

Commit message: FIN
Parts:
- moved R7 53.7 mm to (75.5, 70.0), turned to 45 degrees
- moved R8 52.6 mm to (77.0, 71.0), turned to 45 degrees
- moved C9 49.7 mm to (76.5, 64.0), turned to 135 degrees
- moved C8 45.7 mm to (78.5, 72.2), turned to -135 degrees
- moved C10 44.0 mm to (81.0, 71.8), turned to -90 degrees
- moved C11 43.2 mm to (82.5, 71.8), turned to -90 degrees
- moved C6 3.83 mm to (73.6, 79.0)
- moved C7 3.83 mm to (76.8, 76.5)
- moved U3 3.83 mm to (76.5, 79.0)
- moved C1 3.54 mm to (74.5, 85.5)
- moved C2 3.54 mm to (81.0, 81.0)
- moved U2 3.54 mm to (80.5, 85.5)
- moved R1 1.67 mm to (86.8, 105.0)
- moved R2 1.67 mm to (86.8, 102.5)
- moved U1 1.66 mm to (79.1, 67.0), turned to 135 degrees
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Connections:
- J5 pad 2: VBUS -> +5V
- J5 pad 3: I2S Frame Clock -> I2C_SDA
- J5 pad 4: I2S Bit Clock -> I2C_SCL
- J5 pad 5: I2S D Out -> I2S Frame Clock
- J5 pad 6: I2S D In -> I2S Bit Clock
- J5 pad 7: I2C_SDA -> I2S D Out
- J5 pad 8: I2C_SCL -> I2S D In
- J5 pad 9: +5V -> VBUS
Routing:
- net VBUS: track 0.00 -> 85.0 mm
- net +5V: track 0.00 -> 55.4 mm, vias 0 -> 3
- net +3V3: track 0.00 -> 43.6 mm, vias 0 -> 2
- net I2C_SCL: track 0.00 -> 32.7 mm, vias 0 -> 2
- net I2C_SDA: track 0.00 -> 32.5 mm, vias 0 -> 2
- net Line In L: track 0.00 -> 30.7 mm
- net Line In R: track 0.00 -> 29.5 mm
- net I2S D Out: track 0.00 -> 27.2 mm
- net I2S D In: track 0.00 -> 27.1 mm
- net I2S Frame Clock: track 0.00 -> 26.9 mm
- net I2S Bit Clock: track 0.00 -> 25.9 mm
- net HP_VGND: track 0.00 -> 22.0 mm, vias 0 -> 2
- net HP_R: track 0.00 -> 19.1 mm, vias 0 -> 2
- net Line Out L: track 0.00 -> 18.0 mm
- net Line Out R: track 0.00 -> 17.7 mm
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- added copper zone on B.Cu, net GND
- added copper zone on F.Cu, net GND
