File: PCB FILES/Teensy Synth/Teensy Synth.kicad_sch (KiCad schematic)
At the start: 132 parts, among them J1 Conn_01x09, J2 Conn_01x11_Socket, J2 USB_BOOT, J3 RST, J4 Conn_01x04, SW1 SW_Push, SW10 SW_Push, SW11 SW_Push, SW12 SW_Push, SW13 SW_Push, SW14 SW_Push, SW15 SW_Push, SW16 SW_Push, SW17 SW_Push, SW18 SW_Push, SW19 SW_Push, SW2 SW_Push, SW20 SW_Push, SW21 SW_Push, SW22 SW_Push, SW23 SW_Push, SW24 SW_Push, SW25 SW_Push, SW26 SW_Push, SW27 SW_Push, SW28 SW_Push, SW29 SW_Push, SW3 SW_Push, SW30 SW_Push, SW31 SW_Push, SW32 SW_Push, SW33 SW_Push, SW34 SW_Push, SW35 SW_Push, SW36 SW_Push, SW37 SW_Push, SW38 SW_Push, SW39 SW_Push, SW4 SW_Push, SW40 SW_Push, SW41 SW_Push, SW42 SW_Push, SW43 SW_Push, SW44 SW_Push, SW45 SW_Push, SW46 SW_Push, SW47 SW_Push, SW48 RotaryEncoder, SW49 RotaryEncoder, SW5 SW_Push, SW50 RotaryEncoder, SW51 RotaryEncoder, SW52 RotaryEncoder, SW6 SW_Push, SW7 SW_Push, SW8 SW_Push, SW9 SW_Push, U1 RP2040, U1 Teensy4.1, U2 NCP1117-3.3_SOT223, U2 TPS61090, U3 W25Q128JVS, U6 MCP73871, Y1 Crystal_Small

Commit message: encoder daughterboard
Parts:
- added C16: 10k, symbol Device:C_Small
- added C17: 10uf, symbol Device:C_Small
- added C18: 0.1uf, symbol Device:C_Small
- added L1: 6.8uH, symbol Device:L
- added R10: 100k, symbol Device:R_Small
- added R11, R12: 1k, symbol Device:R_Small
- added R13: 1.87M, symbol Device:R_Small
- added R14: 340K, symbol Device:R_Small
- added R7: 1.0k, symbol Device:R_Small
- added R8: 10k, symbol Device:R_Small
- added R9: 270k, symbol Device:R_Small
Connections:
- net GND: now also U2.10 (SYNC), U2.13 (GND), U6.7 (STAT2), U6.8 (STAT1/~{LBO}), C16.2, C17.2, C18.2, R10.2, R11.2, R12.2, R14.2, R7.2, R8.2
- net VBAT: now also U2.8 (VBAT), U6.1 (OUT), U6.20 (OUT), C17.1, C18.1, L1.1, R13.1; no longer U6.14 (V_{BAT}), U6.15 (V_{BAT}), U6.16 (V_{BAT_SENSE})
- net VUSB: now also U6.17 (CE), U6.3 (SEL), U6.9 (~{TE}), R9.1
- net at U6.12 (PROG3): now also R8.1
- net at U6.13 (PROG1): now also R7.1
- net at U6.2 (VPCC): now also R10.1, R9.2
- net at U2.3 (SW): now also U2.4 (SW), L1.2
- net at U2.9 (LBI): now also R13.2, R14.1
- new net VLIPO: C16.1, U6.14 (V_{BAT}), U6.15 (V_{BAT}), U6.16 (V_{BAT_SENSE})
Other:
- moved on the sheet: R6, U2
